Commit message: Your commit message here

File: install/superbot_description/share/superbot_description/URDF/superbot.urdf.xacro (robot description, xacro)
@@ -12,4 +12,9 @@
     <link name="base_footprint"/>
     <link name="base_link">
+        <inertial>
+            <origin xyz="0 0 0.1" rpy="0 0 0"/>
+            <mass value="5.0"/>
+            <inertia ixx="0.1" ixy="0.0" ixz="0.0" iyy="0.1" iyz="0.0" izz="0.1"/>
+        </inertial>
         <visual>
             <geometry>
@@ -27,4 +32,9 @@
     </link>
     <link name="lidar">
+        <inertial>
+            <origin xyz="0 0 0" rpy="0 0 0"/>
+            <mass value="0.5"/>
+            <inertia ixx="0.01" ixy="0.0" ixz="0.0" iyy="0.01" iyz="0.0" izz="0.01"/>
+        </inertial>
         <visual>
             <geometry>
@@ -43,4 +53,9 @@
     <xacro:macro name="wheel_link" params="prefix">
         <link name="${prefix}_wheel">
+            <inertial>
+                <origin xyz="0 0 0" rpy="0 0 0"/>
+                <mass value="1.0"/>
+                <inertia ixx="0.005" ixy="0.0" ixz="0.0" iyy="0.005" iyz="0.0" izz="0.005"/>
+            </inertial>
             <visual>
                 <geometry>
@@ -61,4 +76,9 @@
     <xacro:wheel_link prefix="right"/>
     <link name="caster_wheel">
+        <inertial>
+            <origin xyz="0 0 0" rpy="0 0 0"/>
+            <mass value="0.2"/>
+            <inertia ixx="0.001" ixy="0.0" ixz="0.0" iyy="0.001" iyz="0.0" izz="0.001"/>
+        </inertial>
         <visual>
             <geometry>
