Commit message: new

File: install/superbot_description/share/superbot_description/URDF/superbot.urdf (robot description, URDF)
Before this commit: robot superbot, 6 links, 5 joints
Links:
- link base_link: mass None -> 5.0
- link caster_wheel: mass None -> 0.2
- link left_wheel: mass None -> 1.0
- link lidar: mass None -> 0.5; geometry collision cylinder length=0.05 radius=0.1; visual cylinder length=0.05 radius=0.1
- link right_wheel: mass None -> 1.0
