Commit message: a

File: src/superbot_description/URDF/superbot.urdf (robot description, URDF)
Before this commit: robot superbot, 6 links, 5 joints
Joints:
- joint base_left_wheel_joint: origin xyz=-0.15 0.225 0 rpy=0 0 0 -> xyz=-0.3 0.225 0 rpy=0 0 0
- joint base_right_wheel_joint: origin xyz=-0.15 -0.225 0 rpy=0 0 0 -> xyz=-0.3 -0.225 0 rpy=0 0 0
