Commit message: Resolved merge conflicts

File: src/superbot_description/URDF/superbot.urdf.xacro (robot description, xacro)
@@ -1,4 +1,4 @@
 <?xml version="1.0"?>
-<robot name="superbot">
+<robot name="superbot" xmlns:xacro="http://www.ros.org/wiki/xacro">
     <material name="red">
         <color rgba="1.0 0.0 0.0 1.0"/>
@@ -41,4 +41,21 @@
         </collision>
     </link>
+    <xacro:macro name="wheel_link" params="prefix">
+        <link name="left_wheel">
+            <visual>
+                <geometry>
+                    <cylinder radius="0.1" length="0.05"/>
+                </geometry>
+                <origin xyz="0 0 0" rpy="1.57 0 0"/>
+                <material name="white"/>
+            </visual>
+            <collision>
+                <geometry>
+                    <cylinder radius="0.1" length="0.05"/>
+                </geometry>
+                <origin xyz="0 0 0" rpy="1.57 0 0"/>
+            </collision>
+        </link>
+    </xacro:macro>
     <link name="left_wheel">
         <visual>

Commit message: Your commit message here

File: src/superbot_description/URDF/superbot.urdf.xacro (robot description, xacro)
@@ -42,5 +42,5 @@
     </link>
     <xacro:macro name="wheel_link" params="prefix">
-        <link name="left_wheel">
+        <link name="${prefix}_wheel">
             <visual>
                 <geometry>
@@ -58,34 +58,6 @@
         </link>
     </xacro:macro>
-    <link name="left_wheel">
-        <visual>
-            <geometry>
-                <cylinder radius="0.1" length="0.05"/>
-            </geometry>
-            <origin xyz="0 0 0" rpy="1.57 0 0"/>
-            <material name="white"/>
-        </visual>
-        <collision>
-            <geometry>
-                <cylinder radius="0.1" length="0.05"/>
-            </geometry>
-            <origin xyz="0 0 0" rpy="1.57 0 0"/>
-        </collision>
-    </link>
-    <link name="right_wheel">
-        <visual>
-            <geometry>
-                <cylinder radius="0.1" length="0.05"/>
-            </geometry>
-            <origin xyz="0 0 0" rpy="1.57 0 0"/>
-            <material name="white"/>
-        </visual>
-        <collision>
-            <geometry>
-                <cylinder radius="0.1" length="0.05"/>
-            </geometry>
-            <origin xyz="0 0 0" rpy="1.57 0 0"/>
-        </collision>
-    </link>
+    <xacro:wheel_link prefix="left"/>
+    <xacro:wheel_link prefix="right"/>
     <link name="caster_wheel">
         <visual>

Commit message: Update superbot.urdf.xacro

File: src/superbot_description/URDF/superbot.urdf.xacro (robot description, xacro)
@@ -1,163 +1,169 @@
 <?xml version="1.0"?>
 <robot name="superbot" xmlns:xacro="http://www.ros.org/wiki/xacro">
-    <!-- Materials -->
-    <material name="red">
-        <color rgba="1.0 0.0 0.0 1.0"/>
-    </material>
-    <material name="green">
-        <color rgba="0 0.6 0 1"/>
-    </material>
-    <material name="white">
-        <color rgba="1 1 1 1"/>
-    </material>
-    <!-- Base Links -->
-    <link name="base_footprint"/>
+    <!-- Body dimensions -->
+    <xacro:property name="body_x" value="1"/>
+    <xacro:property name="body_y" value="0.6"/>
+    <xacro:property name="body_z" value="0.3"/>
+    <!-- Wheel dimensions and locations -->
+    <xacro:property name="wheel_r" value="0.15"/>
+    <xacro:property name="wheel_l" value="0.1"/>
+    <xacro:property name="wheel_z" value="-0.1"/>
+    <!-- Castor wheel dimensions and locations -->
+    <xacro:property name="castor_r" value="0.15"/>
+    <xacro:property name="castor_z" value="-0.1"/>
+    <!-- Material density -->
+    <xacro:property name="body_density" value="2710.0"/>
+    <xacro:property name="wheel_density" value="2710.0"/>
+    <xacro:property name="castor_density" value="2710.0"/>
+    <!-- Pi Value -->
+    <xacro:property name="pi" value="3.14159265"/>
+    <!-- Mass property -->
+    <xacro:property name="body_mass" value="${body_density * body_x * body_y * body_z}"/>
+    <xacro:property name="wheel_mass" value="${wheel_density * pi * wheel_r * wheel_r * wheel_l}"/>
+    <xacro:property name="castor_mass" value="${castor_density * (4.0 / 3.0) * pi * castor_r * castor_r * castor_r}"/>
+    <!-- Moment of Inertia Wheel -->
+    <xacro:property name="Iz_wheel" value="${0.5 * wheel_mass * wheel_r * wheel_r}"/>
+    <xacro:property name="I_wheel" value="${(1.0 / 12.0) * wheel_mass * (3.0 * wheel_r * wheel_r + wheel_l * wheel_l)}"/>
+    <!-- Moment of Inertia Castor Wheel -->
+    <xacro:property name="I_castor" value="${(2.0 / 5.0) * castor_mass * castor_r * castor_r}"/>
+    <!-- Inertial macro for wheel -->
+    <xacro:macro name="inertia_wheel">
+        <inertial>
+            <origin rpy="0 0 0" xyz="0 0 0"/>
+            <mass value="${wheel_mass}"/>
+            <inertia ixx="${I_wheel}" ixy="0.0" ixz="0.0" iyy="${I_wheel}" iyz="0.0" izz="${Iz_wheel}"/>
+        </inertial>
+    </xacro:macro>
+    <!-- Inertial macro for castor wheel -->
+    <xacro:macro name="inertia_castor">
+        <inertial>
+            <origin rpy="0 0 0" xyz="0 0 0"/>
+            <mass value="${castor_mass}"/>
+            <inertia ixx="${I_castor}" ixy="0.0" ixz="0.0" iyy="${I_castor}" iyz="0.0" izz="${I_castor}"/>
+        </inertial>
+    </xacro:macro>
+    <!-- Gazebo Plugin Include -->
+    <xacro:include filename="$(find superbot_description)/URDF/superbot.gazebo.xacro"/>
+    <!-- Define Lidar Properties -->
+    <xacro:property name="lidar_radius" value="0.1"/>
+    <xacro:property name="lidar_length" value="0.3"/>
+    <xacro:property name="lidar_z" value="0.25"/>
+    <!-- Dummy Link and Joint -->
+    <link name="dummy"/>
+    <joint name="dummy_joint" type="fixed">
+        <parent link="dummy"/>
+        <child link="base_link"/>
+    </joint>
+    <!-- Base Link -->
     <link name="base_link">
-        <inertial>
-            <origin xyz="0 0 0.1" rpy="0 0 0"/>
-            <mass value="5.0"/>
-            <inertia ixx="0.1" ixy="0.0" ixz="0.0" iyy="0.1" iyz="0.0" izz="0.1"/>
-        </inertial>
         <visual>
             <geometry>
-                <box size="0.6 0.4 0.2"/>
+                <box size="${body_x} ${body_y} ${body_z}"/>
             </geometry>
-            <origin xyz="0 0 0.1" rpy="0 0 0"/>
-            <material name="green"/>
+            <origin rpy="0 0 0" xyz="0 0 0"/>
         </visual>
         <collision>
             <geometry>
-                <box size="0.6 0.4 0.2"/>
+                <box size="${body_x} ${body_y} ${body_z}"/>
             </geometry>
-            <origin xyz="0 0 0.1" rpy="0 0 0"/>
+            <origin rpy="0 0 0" xyz="0 0 0"/>
         </collision>
+        <inertial>
+            <origin rpy="0 0 0" xyz="0 0 0"/>
+            <mass value="${body_mass}"/>
+            <inertia ixx="${(1 / 12) * body_mass * (body_y * body_y + body_z * body_z)}"
+                     ixy="0"
+                     ixz="0"
+                     iyy="${(1 / 12) * body_mass * (body_x * body_x + body_z * body_z)}"
+                     iyz="0"
+                     izz="${(1 / 12) * body_mass * (body_x * body_x + body_y * body_y)}"/>
+        </inertial>
+    </link>
+    <!-- Wheel Joints and Links -->
+    <!-- Right Wheel -->
+    <joint name="right_joint" type="continuous">
+        <parent link="base_link"/>
+        <child link="right_wheel"/>
+        <origin xyz="${-2 * wheel_r} ${-body_y / 2 - wheel_l / 2} ${wheel_z}" rpy="0 0 0"/>
+        <axis xyz="0 1 0"/>
+    </joint>
+    <link name="right_wheel">
+        <visual>
+            <origin rpy="1.57 0 0" xyz="0 0 0"/>
+            <geometry>
+                <cylinder length="${wheel_l}" radius="${wheel_r}"/>
+            </geometry>
+        </visual>
+        <collision>
+            <origin rpy="1.57 0 0" xyz="0 0 0"/>
+            <geometry>
+                <cylinder length="${wheel_l}" radius="${wheel_r}"/>
+            </geometry>
+        </collision>
+        <xacro:inertia_wheel/>
+    </link>
+    <!-- Left Wheel -->
+    <joint name="left_joint" type="continuous">
+        <parent link="base_link"/>
+        <child link="left_wheel"/>
+        <origin xyz="${-2 * wheel_r} ${body_y / 2 + wheel_l / 2} ${wheel_z}" rpy="0 0 0"/>
+        <axis xyz="0 1 0"/>
+    </joint>
+    <link name="left_wheel">
+        <visual>
+            <origin rpy="1.57 0 0" xyz="0 0 0"/>
+            <geometry>
+                <cylinder length="${wheel_l}" radius="${wheel_r}"/>
+            </geometry>
+        </visual>
+        <collision>
+            <origin rpy="1.57 0 0" xyz="0 0 0"/>
+            <geometry>
+                <cylinder length="${wheel_l}" radius="${wheel_r}"/>
+            </geometry>
+        </collision>
+        <xacro:inertia_wheel/>
+    </link>
+    <!-- Castor Wheel -->
+    <joint name="castor_joint" type="fixed">
+        <parent link="base_link"/>
+        <child link="castor_wheel"/>
+        <origin xyz="${2 * castor_r} 0 ${castor_z}" rpy="0 0 0"/>
+    </joint>
+    <link name="castor_wheel">
+        <visual>
+            <origin rpy="0 0 0" xyz="0 0 0"/>
+            <geometry>
+                <sphere radius="${castor_r}"/>
+            </geometry>
+        </visual>
+        <collision>
+            <origin rpy="0 0 0" xyz="0 0 0"/>
+            <geometry>
+                <sphere radius="${castor_r}"/>
+            </geometry>
+        </collision>
+        <xacro:inertia_castor/>
     </link>
     <!-- Lidar -->
     <link name="lidar">
-        <inertial>
-            <origin xyz="0 0 0" rpy="0 0 0"/>
-            <mass value="0.5"/>
-            <inertia ixx="0.01" ixy="0.0" ixz="0.0" iyy="0.01" iyz="0.0" izz="0.01"/>
-        </inertial>
         <visual>
+            <origin xyz="0 0 ${lidar_z}" rpy="0 0 0"/>
             <geometry>
-                <cylinder radius="0.1" length="0.05"/>
+                <cylinder radius="${lidar_radius}" length="${lidar_length}"/>
             </geometry>
-            <origin xyz="0 0 0" rpy="0 0 0"/>
             <material name="red"/>
         </visual>
         <collision>
+            <origin xyz="0 0 ${lidar_z}" rpy="0 0 0"/>
             <geometry>
-                <box size="0.2 0.2 0.05"/>
+                <cylinder radius="${lidar_radius}" length="${lidar_length}"/>
             </geometry>
-            <origin xyz="0 0 0" rpy="0 0 0"/>
         </collision>
     </link>
-    <!-- Gazebo Lidar Plugin -->
-    <gazebo reference="lidar">
-        <sensor type="ray" name="laser">
-            <pose>0 0 0 0 0 0</pose>
-            <visualize>true</visualize>
-            <update_rate>30</update_rate>
-            <ray>
-                <scan>
-                    <horizontal>
-                        <samples>360</samples>
-                        <resolution>1</resolution>
-                        <min_angle>-1.5708</min_angle>
-                        <max_angle>1.5708</max_angle>
-                    </horizontal>
-                </scan>
-                <range>
-                    <min>0.1</min>
-                    <max>10.0</max>
-                    <resolution>0.01</resolution>
-                </range>
-                <noise>
-                    <type>gaussian</type>
-                    <mean>0.0</mean>
-                    <stddev>0.01</stddev>
-                </noise>
-            </ray>
-            <plugin name="gazebo_ros_laser" filename="libgazebo_ros_laser.so">
-                <topicName>/scan</topicName>
-                <frameName>lidar</frameName>
-            </plugin>
-        </sensor>
-    </gazebo>
-    <!-- Wheels -->
-    <xacro:macro name="wheel_link" params="prefix">
-        <link name="${prefix}_wheel">
-            <inertial>
-                <origin xyz="0 0 0" rpy="0 0 0"/>
-                <mass value="1.0"/>
-                <inertia ixx="0.005" ixy="0.0" ixz="0.0" iyy="0.005" iyz="0.0" izz="0.005"/>
-            </inertial>
-            <visual>
-                <geometry>
-                    <cylinder radius="0.1" length="0.05"/>
-                </geometry>
-                <origin xyz="0 0 0" rpy="1.57 0 0"/>
-                <material name="white"/>
-            </visual>
-            <collision>
-                <geometry>
-                    <cylinder radius="0.1" length="0.05"/>
-                </geometry>
-                <origin xyz="0 0 0" rpy="1.57 0 0"/>
-            </collision>
-        </link>
-    </xacro:macro>
-    <!-- Instantiate Wheels -->
-    <xacro:wheel_link prefix="left"/>
-    <xacro:wheel_link prefix="right"/>
-    <!-- Caster Wheel -->
-    <link name="caster_wheel">
-        <inertial>
-            <origin xyz="0 0 0" rpy="0 0 0"/>
-            <mass value="0.2"/>
-            <inertia ixx="0.001" ixy="0.0" ixz="0.0" iyy="0.001" iyz="0.0" izz="0.001"/>
-        </inertial>
-        <visual>
-            <geometry>
-                <sphere radius="0.05"/>
-            </geometry>
-            <origin xyz="0 0 0" rpy="0 0 0"/>
-            <material name="white"/>
-        </visual>
-        <collision>
-            <geometry>
-                <sphere radius="0.05"/>
-            </geometry>
-            <origin xyz="0 0 0" rpy="0 0 0"/>
-        </collision>
-    </link>
-    <!-- Joints -->
-    <joint name="base_joint" type="fixed">
-        <parent link="base_footprint"/>
-        <child link="base_link"/>
-        <origin xyz="0 0 0.1" rpy="0 0 0"/>
-    </joint>
-    <joint name="base_lidar_joint" type="fixed">
+    <joint name="lidar_joint" type="fixed">
         <parent link="base_link"/>
         <child link="lidar"/>
-        <origin xyz="0 0 0.225" rpy="0 0 0"/>
-    </joint>
-    <joint name="base_left_wheel_joint" type="continuous">
-        <parent link="base_link"/>
-        <child link="left_wheel"/>
-        <origin xyz="-0.15 0.225 0" rpy="0 0 0"/>
-        <axis xyz="0 1 0"/>
-    </joint>
-    <joint name="base_right_wheel_joint" type="continuous">
-        <parent link="base_link"/>
-        <child link="right_wheel"/>
-        <origin xyz="-0.15 -0.225 0" rpy="0 0 0"/>
-        <axis xyz="0 1 0"/>
-    </joint>
-    <joint name="base_caster_wheel_joint" type="fixed">
-        <parent link="base_link"/>
-        <child link="caster_wheel"/>
-        <origin xyz="0.2 0 -0.05" rpy="0 0 0"/>
+        <origin xyz="0 0 ${lidar_z}" rpy="0 0 0"/>
     </joint>
 </robot>
